File: pcb/Env-Sensors-1.kicad_sch (KiCad schematic)
At the start: 15 parts, among them J1 SEN66, U11 SGP41, U12 SCD41, U16 SHT45

Commit message: Rev A Updates
Support LD2410S and LD2420 Radars in same connector as C4001. Now using 3.3V instead of 5V.
Removed Power control for Radars.
Added DS18S20 to measure CO sensor temperature directly.
Reworked SHT4X layout to reduce thermal transfer.
Parts:
- renumbered C28 to C24, C29 to C25, C30 to C26, C31 to C27, C34 to C30, C38 to C34, C40 to C36, C43 to C39, R16 to R14, R23 to R17, R22 to R18, U12 to U10, U16 to U14, U11 to U9
Changed lines of the file:
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@@
 	(title_block
 		(title "ESPHome Parking Assistant")
-		(date "2025-04-18")
-		(rev "A")
+		(date "2025-09-23")
+		(rev "B")
 		(company "Mike Lawrence")
 	)
@@
 		(on_board yes)
 		(dnp no)
-		(property "Reference" "C30"
+		(property "Reference" "C26"
 			(at 153.67 75.184 0)
 			(effects
@@
 			(project "ESPHome-Indoor-Multi-Sensor"
 				(path "/e74956a0-c576-42e7-be96-7ce5c3135988/c3a2a756-5acc-4a4f-a61d-07af630c1ef7"
-					(reference "C30")
+					(reference "C26")
 					(unit 1)
 				)
@@
 		(on_board yes)
 		(dnp no)
-		(property "Reference" "C34"
+		(property "Reference" "C30"
 			(at 201.93 76.454 0)
 			(effects
@@
 			(project "ESPHome-Indoor-Multi-Sensor"
 				(path "/e74956a0-c576-42e7-be96-7ce5c3135988/c3a2a756-5acc-4a4f-a61d-07af630c1ef7"
-					(reference "C34")
+					(reference "C30")
 					(unit 1)
 				)
@@
 		(on_board yes)
 		(dnp yes)
-		(property "Reference" "R22"
+		(property "Reference" "R18"
 			(at 224.536 121.158 0)
 			(effects
@@
 			(project "ESPHome-Indoor-Multi-Sensor"
 				(path "/e74956a0-c576-42e7-be96-7ce5c3135988/c3a2a756-5acc-4a4f-a61d-07af630c1ef7"
-					(reference "R22")
+					(reference "R18")
 					(unit 1)
 				)
@@
 		(on_board yes)
 		(dnp no)
-		(property "Reference" "C38"
+		(property "Reference" "C34"
 			(at 228.6 52.07 90)
 			(effects
@@
 			(project "ESPHome-Indoor-Multi-Sensor"
 				(path "/e74956a0-c576-42e7-be96-7ce5c3135988/c3a2a756-5acc-4a4f-a61d-07af630c1ef7"
-					(reference "C38")
+					(reference "C34")
 					(unit 1)
 				)
@@
 		(on_board yes)
 		(dnp no)
-		(property "Reference" "U11"
+		(property "Reference" "U9"
 			(at 122.936 69.85 0)
 			(effects
@@
 			(project "ESPHome-Indoor-Multi-Sensor"
 				(path "/e74956a0-c576-42e7-be96-7ce5c3135988/c3a2a756-5acc-4a4f-a61d-07af630c1ef7"
-					(reference "U11")
+					(reference "U9")
 					(unit 1)
 				)
@@
 		(on_board yes)
 		(dnp no)
-		(property "Reference" "C40"
+		(property "Reference" "C36"
 			(at 228.6 77.47 90)
 			(effects
@@
 			(project "ESPHome-Indoor-Multi-Sensor"
 				(path "/e74956a0-c576-42e7-be96-7ce5c3135988/c3a2a756-5acc-4a4f-a61d-07af630c1ef7"
-					(reference "C40")
+					(reference "C36")
 					(unit 1)
 				)
@@
 		(on_board yes)
 		(dnp no)
-		(property "Reference" "C31"
+		(property "Reference" "C27"
 			(at 143.51 75.184 0)
 			(effects
@@
 			(project "ESPHome-Indoor-Multi-Sensor"
 				(path "/e74956a0-c576-42e7-be96-7ce5c3135988/c3a2a756-5acc-4a4f-a61d-07af630c1ef7"
-					(reference "C31")
+					(reference "C27")
 					(unit 1)
 				)
@@
 		(on_board yes)
 		(dnp no)
-		(property "Reference" "C29"
+		(property "Reference" "C25"
 			(at 68.58 103.378 90)
 			(effects
@@
 			(project "ESPHome-Indoor-Multi-Sensor"
 				(path "/e74956a0-c576-42e7-be96-7ce5c3135988/c3a2a756-5acc-4a4f-a61d-07af630c1ef7"
-					(reference "C29")
+					(reference "C25")
 					(unit 1)
 				)
@@
 		(on_board yes)
 		(dnp no)
-		(property "Reference" "U16"
+		(property "Reference" "U14"
 			(at 67.056 59.944 0)
 			(effects
@@
 			(project "ESPHome-Indoor-Multi-Sensor"
 				(path "/e74956a0-c576-42e7-be96-7ce5c3135988/c3a2a756-5acc-4a4f-a61d-07af630c1ef7"
-					(reference "U16")
+					(reference "U14")
 					(unit 1)
 				)
@@
 		(on_board yes)
 		(dnp yes)
-		(property "Reference" "R23"
+		(property "Reference" "R17"
 			(at 214.376 121.158 0)
 			(effects
@@
 			(project "ESPHome-Indoor-Multi-Sensor"
 				(path "/e74956a0-c576-42e7-be96-7ce5c3135988/c3a2a756-5acc-4a4f-a61d-07af630c1ef7"
-					(reference "R23")
+					(reference "R17")
 					(unit 1)
 				)
@@
 		(on_board yes)
 		(dnp no)
-		(property "Reference" "C28"
+		(property "Reference" "C24"
 			(at 81.28 103.124 90)
 			(effects
@@
 			(project "ESPHome-Indoor-Multi-Sensor"
 				(path "/e74956a0-c576-42e7-be96-7ce5c3135988/c3a2a756-5acc-4a4f-a61d-07af630c1ef7"
-					(reference "C28")
+					(reference "C24")
 					(unit 1)
 				)
@@
 		(on_board yes)
 		(dnp no)
-		(property "Reference" "U12"
+		(property "Reference" "U10"
 			(at 78.232 116.84 0)
 			(effects
@@
 			(project "ESPHome-Indoor-Multi-Sensor"
 				(path "/e74956a0-c576-42e7-be96-7ce5c3135988/c3a2a756-5acc-4a4f-a61d-07af630c1ef7"
-					(reference "U12")
+					(reference "U10")
 					(unit 1)
 				)
@@
 		(on_board yes)
 		(dnp no)
-		(property "Reference" "R16"
+		(property "Reference" "R14"
 			(at 127.254 58.42 0)
 			(effects
@@
 			(project "ESPHome-Indoor-Multi-Sensor"
 				(path "/e74956a0-c576-42e7-be96-7ce5c3135988/c3a2a756-5acc-4a4f-a61d-07af630c1ef7"
-					(reference "R16")
+					(reference "R14")
 					(unit 1)
 				)
@@
 		(on_board yes)
 		(dnp no)
-		(property "Reference" "C43"
+		(property "Reference" "C39"
 			(at 81.28 52.324 90)
 			(effects
@@
 			(project "ESPHome-Indoor-Multi-Sensor"
 				(path "/e74956a0-c576-42e7-be96-7ce5c3135988/c3a2a756-5acc-4a4f-a61d-07af630c1ef7"
-					(reference "C43")
+					(reference "C39")
 					(unit 1)
 				)

Commit message: Cleanup schematic, BOM and update gerber files
Parts:
- added R6, R7: 5.1KΩ, Resistor_SMD:R_0402_1005Metric, symbol Device:R
Connections:
- net SCL1: now also R7.2
- net SDA1: now also R6.2
- new net +3.3V: R6.1, R7.1
Other:
- note added: "I^{2}C1 Pullup"
- moved on the sheet: C24, C25, C26, C27, R14, R17, R18, U10, U9
