File: pcb/ESPHome-Indoor-Multi-Sensor.kicad_sch (KiCad schematic)
At the start: 11 parts, among them J2 USB-C, U9 INA228

Commit message: Rev A Updates
Support LD2410S and LD2420 Radars in same connector as C4001. Now using 3.3V instead of 5V.
Removed Power control for Radars.
Added DS18S20 to measure CO sensor temperature directly.
Reworked SHT4X layout to reduce thermal transfer.
Parts:
- renumbered C24 to C20, R12 to R10, R10 to R8, R11 to R9, U9 to U7
Other:
- sheet ESP32-S3 ports: added 1Wire, RDRA_OUT, RDRA_SIG1, RDRA_SIG2, RDRB_OUT, RDRB_RX, RDRB_TX; removed LD24X0_OUT, LD24X0_RX, LD24X0_TX, SEN0609_OUT, SEN0609_RX, SEN0609_TX
- sheet Environmental Sensors 2 ports: added 1Wire; removed none
- sheet Presence Sensors ports: added RDRA_OUT, RDRA_SIG1, RDRA_SIG2, RDRB_OUT, RDRB_RX, RDRB_TX; removed LD24X0_EN, LD24X0_OUT, LD24X0_RX, LD24X0_TX, SEN0609_EN, SEN0609_OUT, SEN0609_RX, SEN0609_TX

Commit message: Add new ina228 to other power supplies
Not finished
Parts:
- removed R10, R8: 10Ω, Resistor_SMD:R_0402_1005Metric, symbol Device:R
- R9: footprint Resistor_SMD:R_1210_3225Metric -> Resistor_SMD:R_0805_2012Metric
Connections:
- net +5V: now also U7.9 (Vin-)
- net VBUS: now also U7.10 (Vin+)
Changed lines of the file:
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@@
 	(wire
 		(pts
-			(xy 140.97 81.28) (xy 140.97 63.5)
+			(xy 140.97 31.75) (xy 140.97 81.28)
 		)
 		(stroke
@@
 	(wire
 		(pts
-			(xy 128.27 55.88) (xy 128.27 31.75)
+			(xy 128.27 31.75) (xy 128.27 78.74)
 		)
 		(stroke
@@
 	(wire
 		(pts
-			(xy 140.97 55.88) (xy 140.97 31.75)
-		)
-		(stroke
-			(width 0)
-			(type default)
-		)
-	)
-	(wire
-		(pts
 			(xy 76.2 49.53) (xy 87.63 49.53)
 		)
@@
 		(pts
 			(xy 139.7 123.19) (xy 195.58 123.19)
-		)
-		(stroke
-			(width 0)
-			(type default)
-		)
-	)
-	(wire
-		(pts
-			(xy 128.27 78.74) (xy 128.27 63.5)
 		)
 		(stroke
@@
 	(symbol
 		(lib_id "Device:R")
-		(at 128.27 59.69 0)
-		(unit 1)
-		(exclude_from_sim no)
-		(in_bom yes)
-		(on_board yes)
-		(dnp no)
-		(property "Reference" "R10"
-			(at 129.54 58.674 0)
-			(effects
-				(font
-					(size 1.27 1.27)
-				)
-				(justify left)
-			)
-		)
-		(property "Value" "10Ω"
-			(at 129.54 60.96 0)
-			(effects
-				(font
-					(size 1.27 1.27)
-				)
-				(justify left)
-			)
-		)
-		(property "Footprint" "Resistor_SMD:R_0402_1005Metric"
-			(at 126.492 59.69 90)
-			(effects
-				(font
-					(size 1.27 1.27)
-				)
-				(hide yes)
-			)
-		)
-		(property "Datasheet" "~"
-			(at 128.27 59.69 0)
-			(effects
-				(font
-					(size 1.27 1.27)
-				)
-				(hide yes)
-			)
-		)
-		(property "Description" "Resistor, 10Ω, 62.5mW, 1%, 0402"
-			(at 128.27 59.69 0)
-			(effects
-				(font
-					(size 1.27 1.27)
-				)
-				(hide yes)
-			)
-		)
-		(property "Manufacturer" "Vishay / Dale"
-			(at 128.27 59.69 0)
-			(effects
-				(font
-					(size 1.27 1.27)
-				)
-				(hide yes)
-			)
-		)
-		(property "Part Number" "CRCW040210R0FKEE"
-			(at 128.27 59.69 0)
-			(effects
-				(font
-					(size 1.27 1.27)
-				)
-				(hide yes)
-			)
-		)
-		(pin "1"
-		)
-		(pin "2"
-		)
-		(instances
-			(project "ESPHome-Indoor-Multi-Sensor"
-				(path "/e74956a0-c576-42e7-be96-7ce5c3135988"
-					(reference "R10")
-					(unit 1)
-				)
-			)
-		)
-	)
-	(symbol
-		(lib_id "Device:R")
 		(at 93.98 73.66 0)
 		(unit 1)
@@
 				(path "/e74956a0-c576-42e7-be96-7ce5c3135988"
 					(reference "#PWR08")
-					(unit 1)
-				)
-			)
-		)
-	)
-	(symbol
-		(lib_id "Device:R")
-		(at 140.97 59.69 0)
-		(mirror y)
-		(unit 1)
-		(exclude_from_sim no)
-		(in_bom yes)
-		(on_board yes)
-		(dnp no)
-		(property "Reference" "R8"
-			(at 139.7 58.674 0)
-			(effects
-				(font
-					(size 1.27 1.27)
-				)
-				(justify left)
-			)
-		)
-		(property "Value" "10Ω"
-			(at 139.7 60.96 0)
-			(effects
-				(font
-					(size 1.27 1.27)
-				)
-				(justify left)
-			)
-		)
-		(property "Footprint" "Resistor_SMD:R_0402_1005Metric"
-			(at 142.748 59.69 90)
-			(effects
-				(font
-					(size 1.27 1.27)
-				)
-				(hide yes)
-			)
-		)
-		(property "Datasheet" "~"
-			(at 140.97 59.69 0)
-			(effects
-				(font
-					(size 1.27 1.27)
-				)
-				(hide yes)
-			)
-		)
-		(property "Description" "Resistor, 10Ω, 62.5mW, 1%, 0402"
-			(at 140.97 59.69 0)
-			(effects
-				(font
-					(size 1.27 1.27)
-				)
-				(hide yes)
-			)
-		)
-		(property "Manufacturer" "Vishay / Dale"
-			(at 140.97 59.69 0)
-			(effects
-				(font
-					(size 1.27 1.27)
-				)
-				(hide yes)
-			)
-		)
-		(property "Part Number" "CRCW040210R0FKEE"
-			(at 140.97 59.69 0)
-			(effects
-				(font
-					(size 1.27 1.27)
-				)
-				(hide yes)
-			)
-		)
-		(pin "1"
-		)
-		(pin "2"
-		)
-		(instances
-			(project "ESPHome-Indoor-Multi-Sensor"
-				(path "/e74956a0-c576-42e7-be96-7ce5c3135988"
-					(reference "R8")
 					(unit 1)
 				)
@@
 			)
 		)
-		(property "Footprint" "Resistor_SMD:R_1210_3225Metric"
+		(property "Footprint" "Resistor_SMD:R_0805_2012Metric"
 			(at 134.62 29.972 90)
 			(effects

Commit message: Rev B Updates finish adding power monitors for 3.3V and 3.3VA
Removed speaker gain jumper
Parts:
- R9: Manufacturer Panasonic -> Vishay; Part Number ERJ-14BSFR15U -> WSL0805R1500FEA18
Other:
- sheet ESP32-S3 ports: added none; removed LD24X0_EN, SEN0609_EN
- sheet Power Supplies ports: added SCL1, SDA1; removed none
- note added: "USB-C Power Measurement"
- note removed: "Power Measurement"
- title: ESPHome Parking Assistant -> ESPHome Indoor Multi-Sensor
Changed lines of the file:
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@@
 	(generator "eeschema")
 	(generator_version "9.0")
-	(paper "A4")
+	(paper "A")
 	(title_block
-		(title "ESPHome Parking Assistant")
-		(date "2025-09-23")
+		(title "ESPHome Indoor Multi-Sensor")
+		(date "2025-09-24")
 		(rev "B")
 		(company "Mike Lawrence")
@@
 		)
 	)
-	(text "Power\nMeasurement"
+	(text "USB-C Power\nMeasurement"
 		(exclude_from_sim no)
-		(at 156.972 43.434 0)
+		(at 159.512 25.908 0)
 		(effects
 			(font
@@
 	(wire
 		(pts
+			(xy 67.31 132.08) (xy 101.6 132.08)
+		)
+		(stroke
+			(width 0)
+			(type default)
+		)
+	)
+	(wire
+		(pts
 			(xy 187.96 76.2) (xy 187.96 102.87)
 		)
@@
 	(wire
 		(pts
+			(xy 67.31 134.62) (xy 101.6 134.62)
+		)
+		(stroke
+			(width 0)
+			(type default)
+		)
+	)
+	(wire
+		(pts
 			(xy 90.17 44.45) (xy 90.17 119.38)
 		)
@@
 		)
 		(column_widths 25.4 25.4)
-		(row_heights 3.81 2.54 2.54 2.54 2.54 2.54 2.54 2.54 2.54)
+		(row_heights 3.81 2.54 2.54 2.54 2.54 2.54 2.54 2.54 2.54 2.54 2.54)
 		(cells
 			(table_cell "Device"
@@
 				)
 			)
-			(table_cell "INA228"
+			(table_cell "INA228 USB-C"
 				(exclude_from_sim no)
 				(at 203.2 31.75 0)
@@
 				)
 			)
-			(table_cell "SHT45"
+			(table_cell "INA228 +3.3V"
 				(exclude_from_sim no)
 				(at 203.2 34.29 0)
@@
 				)
 			)
-			(table_cell "0x44"
+			(table_cell "0x42"
 				(exclude_from_sim no)
 				(at 228.6 34.29 0)
@@
 				)
 			)
-			(table_cell "BMP581"
+			(table_cell "INA228 +3.3VA"
 				(exclude_from_sim no)
 				(at 203.2 36.83 0)
@@
 				)
 			)
-			(table_cell "0x47"
+			(table_cell "0x43"
 				(exclude_from_sim no)
 				(at 228.6 36.83 0)
@@
 				)
 			)
-			(table_cell "CO ADC"
+			(table_cell "SHT45"
 				(exclude_from_sim no)
 				(at 203.2 39.37 0)
@@
 				)
 			)
-			(table_cell "0x48"
+			(table_cell "0x44"
 				(exclude_from_sim no)
 				(at 228.6 39.37 0)
@@
 				)
 			)
-			(table_cell "SGP41"
+			(table_cell "BMP581"
 				(exclude_from_sim no)
 				(at 203.2 41.91 0)
@@
 				)
 			)
-			(table_cell "0x59"
+			(table_cell "0x47"
 				(exclude_from_sim no)
 				(at 228.6 41.91 0)
@@
 				)
 			)
-			(table_cell "SCD41"
+			(table_cell "CO ADC"
 				(exclude_from_sim no)
 				(at 203.2 44.45 0)
@@
 				)
 			)
-			(table_cell "0x62"
+			(table_cell "0x48"
 				(exclude_from_sim no)
 				(at 228.6 44.45 0)
@@
 				)
 			)
-			(table_cell "SEN66"
+			(table_cell "SGP41"
 				(exclude_from_sim no)
 				(at 203.2 46.99 0)
@@
 				)
 			)
-			(table_cell "0x6B"
+			(table_cell "0x59"
 				(exclude_from_sim no)
 				(at 228.6 46.99 0)
@@
 				)
 			)
+			(table_cell "SCD41"
+				(exclude_from_sim no)
+				(at 203.2 49.53 0)
+				(size 25.4 2.54)
+				(margins 0.9525 0.9525 0.9525 0.9525)
+				(span 1 1)
+				(fill
+					(type none)
+				)
+				(effects
+					(font
+						(size 1.27 1.27)
+					)
+					(justify left)
+				)
+			)
+			(table_cell "0x62"
+				(exclude_from_sim no)
+				(at 228.6 49.53 0)
+				(size 25.4 2.54)
+				(margins 0.9525 0.9525 0.9525 0.9525)
+				(span 1 1)
+				(fill
+					(type none)
+				)
+				(effects
+					(font
+						(size 1.27 1.27)
+					)
+				)
+			)
+			(table_cell "SEN66"
+				(exclude_from_sim no)
+				(at 203.2 52.07 0)
+				(size 25.4 2.54)
+				(margins 0.9525 0.9525 0.9525 0.9525)
+				(span 1 1)
+				(fill
+					(type none)
+				)
+				(effects
+					(font
+						(size 1.27 1.27)
+					)
+					(justify left)
+				)
+			)
+			(table_cell "0x6B"
+				(exclude_from_sim no)
+				(at 228.6 52.07 0)
+				(size 25.4 2.54)
+				(margins 0.9525 0.9525 0.9525 0.9525)
+				(span 1 1)
+				(fill
+					(type none)
+				)
+				(effects
+					(font
+						(size 1.27 1.27)
+					)
+				)
+			)
 		)
 	)
@@
 			)
 		)
-		(property "Description" "Current Sense Resistor, 150mΩ, 500mW, 1%, 1210"
+		(property "Description" "Current Sense Resistor, 150mΩ, 250mW, 1%, 75ppm, 0805"
 			(at 134.62 31.75 0)
 			(effects
@@
 			)
 		)
-		(property "Manufacturer" "Panasonic"
+		(property "Manufacturer" "Vishay"
 			(at 134.62 31.75 0)
 			(effects
@@
 			)
 		)
-		(property "Part Number" "ERJ-14BSFR15U"
+		(property "Part Number" "WSL0805R1500FEA18"
 			(at 134.62 31.75 0)
 			(effects
@@
 			)
 		)
+		(pin "SCL1" input
+			(at 67.31 134.62 0)
+			(effects
+				(font
+					(size 1.27 1.27)
+				)
+				(justify right)
+			)
+		)
+		(pin "SDA1" bidirectional
+			(at 67.31 132.08 0)
+			(effects
+				(font
+					(size 1.27 1.27)
+				)
+				(justify right)
+			)
+		)
 		(instances
 			(project "ESPHome-Indoor-Multi-Sensor"
@@
 			)
 		)
-		(pin "LD24X0_EN" output
+		(pin "SDA1" bidirectional
 			(at 101.6 132.08 180)
 			(effects
@@
 			)
 		)
-		(pin "SEN0609_EN" output
-			(at 101.6 129.54 180)
+		(pin "SCL1" output
+			(at 101.6 134.62 180)
 			(effects
 				(font
