File: pcb/ESPHome-Indoor-Multi-Sensor.kicad_sch (KiCad schematic)
At the start: 9 parts, among them J2 USB-C, U7 INA228

Commit message: BOM Updates
No PCB changes. This is still Rev.B
Other:
- note added: "USB-C Energy Measurement"
- note removed: "USB-C Power Measurement"
Changed lines of the file:
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@@
 		)
 	)
-	(text "USB-C Power\nMeasurement"
+	(text "USB-C Energy\nMeasurement"
 		(exclude_from_sim no)
 		(at 159.512 25.908 0)
@@
 				)
 			)
-			(table_cell "INA228 +3.3V"
+			(table_cell "INA238 +3.3V"
 				(exclude_from_sim no)
 				(at 203.2 34.29 0)
@@
 				)
 			)
-			(table_cell "INA228 +3.3VA"
+			(table_cell "INA238 +3.3VA"
 				(exclude_from_sim no)
 				(at 203.2 36.83 0)
@@
 			)
 		)
-		(property "Description" "IC, High-Side or Low-Side Measurement, Bi-Directional Current and Power Monitor (0-85V) with I2C, SMBus-, and PMBus-Compatible Interface, VSSOP-10"
+		(property "Description" "IC, 85-V, 20-Bit, Ultra-Precise Power-Energy-Charge Monitor With I2C Interface, VSSOP-10"
 			(at 160.02 76.2 0)
 			(effects

Commit message: Design now uses one ina228 and two ina232 power sensors
Reduces cost without sacrificing functionality. Mainly wanted power supply voltage and currents.
Other:
- sheet ESP32-S3 ports: added 1WIRE; removed 1Wire
- sheet Environmental Sensors 2 ports: added 1WIRE; removed 1Wire
Changed lines of the file:
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@@
 		)
 	)
-	(label "1Wire"
+	(label "1WIRE"
 		(at 146.05 125.73 0)
 		(effects
@@
 			)
 		)
-		(pin "1Wire" bidirectional
+		(pin "1WIRE" bidirectional
 			(at 203.2 107.95 180)
 			(effects
@@
 			)
 		)
-		(pin "1Wire" bidirectional
+		(pin "1WIRE" bidirectional
 			(at 139.7 125.73 0)
 			(effects
