File: pcb/ESP32.kicad_sch (KiCad schematic)
At the start: 28 parts, among them J5 SPKR, SW1 BOOT, SW2 RESET, U1 SN74LV1T34DBV, U3 MAX98357A, U6 ESP32-S3-WROOM-2-N32R16V

Commit message: BOM Updates
No PCB changes. This is still Rev.B
Connections:
- net 1Wire renamed 1WIRE
Changed lines of the file:
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@@
 		)
 	)
-	(hierarchical_label "1Wire"
+	(hierarchical_label "1WIRE"
 		(shape bidirectional)
 		(at 101.6 73.66 0)
