File: pcb/stencil/stencil.kicad_pcb (KiCad board)
At the start: 4 copper layers, 52.5 x 59.7 mm, 110 parts, among them J1 SEN66, J2 USB-C, J3 SEN0609, J4 LD2410, J5 SPKR, J6 LD2450, Q1 MMBFJ201, SW1 BOOT, SW2 RESET, T1 Tab, T10 Tab, T2 Tab, T3 Tab, T4 Tab, T5 Tab, T6 Tab, T7 Tab, T8 Tab, T9 Tab, U1 SN74LV1T34DBV, U10 SCD41, U11 BMP581, U12 MCP6042, U13 ADS1115, U14 SHT45, U15 EKMC1603111, U16 TGS5141, U17 DS18S20, U2 TLV62568DRL, U3 MAX98357A, U4 TLV75533PDRV, U5 TLV62568DRL, U6 ESP32-S3-WROOM-2-N32R16V, U7 INA228, U8 TSL2591, U9 SGP41

Commit message: Rev B Updates finish adding power monitors for 3.3V and 3.3VA
Removed speaker gain jumper
Parts:
- removed JP1: Gain, TMM-105-01-X-D-SM:SAMTEC_TMM-105-01-X-D-SM
- added C40: 100nF, Capacitor_SMD:C_0402_1005Metric, F.Cu at (109.5, 57.3)
- added C41: 100nF, Capacitor_SMD:C_0402_1005Metric, F.Cu at (112.3, 50.4)
- added U18: INA228, Package_SO:VSSOP-10_3x3mm_P0.5mm, F.Cu at (107.2, 59.0)
- added U19: INA228, Package_SO:VSSOP-10_3x3mm_P0.5mm, F.Cu at (110.1, 52.1)
- R10: value 10Ω -> 80mΩ; footprint Resistor_SMD:R_0402_1005Metric -> Resistor_SMD:R_0603_1608Metric
- R8: value 10Ω -> 68mΩ; footprint Resistor_SMD:R_0402_1005Metric -> Resistor_SMD:R_0603_1608Metric
- R9: footprint Resistor_SMD:R_1210_3225Metric -> Resistor_SMD:R_0805_2012Metric
- moved R10 13.3 mm to (109.4, 48.2)
- moved R11 12.4 mm to (117.6, 48.8)
- moved R8 5.81 mm to (106.5, 55.1)
- moved C20 5.24 mm to (102.2, 61.2)
- moved R7 4.61 mm to (112.3, 55.9), turned to 180 degrees
- moved R6 4.39 mm to (112.3, 56.9), turned to 180 degrees
- moved U7 4.32 mm to (101.5, 59.0)
- moved R1 3.80 mm to (100.8, 42.2)
- moved C15 2.87 mm to (110.7, 45.1)
- moved C14 2.86 mm to (110.6, 46.2), turned to 180 degrees
- moved R9 1.79 mm to (97.3, 59.7)
Connections:
- net +3.6V renamed /Power Supplies/+3.6V_SRC
- C14 pad 2: +3.3VA -> /Power Supplies/+3.3VA_SRC
- C15 pad 1: +3.3VA -> /Power Supplies/+3.3VA_SRC
- C17 pad 2: +3.3V -> /Power Supplies/+3.3V_SRC
- C18 pad 1: +3.3V -> /Power Supplies/+3.3V_SRC
- C19 pad 1: +3.3V -> /Power Supplies/+3.3V_SRC
- L2 pad 2: +3.3V -> /Power Supplies/+3.3V_SRC
- R10 pad 1: /VBUS -> /Power Supplies/+3.3VA_SRC
- R10 pad 2: Net-(U7-Vin+) -> +3.3VA
- R11 pad 1: Net-(JP1-Pin_10) -> GND
- R4 pad 1: +3.3V -> /Power Supplies/+3.3V_SRC
- R8 pad 1: +5V -> /Power Supplies/+3.3V_SRC
- R8 pad 2: Net-(U7-Vin-) -> +3.3V
- U4 pad 1: +3.3VA -> /Power Supplies/+3.3VA_SRC
- U7 pad 10: Net-(U7-Vin+) -> /VBUS
- U7 pad 9: Net-(U7-Vin-) -> +5V
Routing:
- net +5V: track 46.3 -> 24.4 mm, vias 32 -> 33
- net Net-(U3-GAIN_SLOT): track 19.7 -> 1.91 mm, vias 2 -> 0
- net Net-(JP1-Pin_10): track 15.8 -> 0.00 mm
- net /Power Supplies/+3.3V_SRC: track 0.00 -> 15.3 mm, vias 0 -> 2
- net +3.3VA: track 115.7 -> 125.4 mm
- net /SCL1: track 115.3 -> 123.6 mm
- net /Power Supplies/+3.3VA_SRC: track 0.00 -> 6.74 mm
- net +3.3V: track 17.5 -> 13.5 mm, vias 19 -> 20
- net Net-(U7-Vin-): track 3.67 -> 0.00 mm
- net Net-(U2-FB): track 5.75 -> 2.20 mm, vias 2 -> 0
- net /Power Supplies/+3.6V_SRC: track 4.92 -> 8.45 mm
- net GND: track 162.0 -> 165.2 mm, vias 78 -> 85
- net Net-(U7-Vin+): track 3.17 -> 0.00 mm
- net /VBUS: track 13.4 -> 10.5 mm, vias 22 -> 24
- net /SDA1: track 119.7 -> 120.8 mm
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- added copper zone on F.Cu, net /Power Supplies/+3.3VA_SRC
- added copper zone on F.Cu, net /Power Supplies/+3.3V_SRC
Other:
- board text added: "HUMIDITY"
- board text added: "REV B 2025-09-24"
- board text removed: "12dB"
- board text removed: "15dB"
- board text removed: "3dB"
- board text removed: "6dB"
- board text removed: "9dB"
- board text removed: "HMD"
- board text removed: "REV B 2025-09-22"
- board text removed: "SPKR Gain"
